Commit message: ik solver

File: src/mearm_common/urdf/mearm.urdf (robot description, URDF)
Before this commit: robot mearm, 3 links, 2 joints
Links:
- removed link link2
- added link base; visual cylinder length=0.6 radius=0.2
- link link1: mass 1 -> None; geometry visual box size=0.6 0.1 0.2
Joints:
- joint base: child link1 -> base
- joint left: child link2 -> link1; origin xyz=0 0 0.5 rpy=0 0 3.1416 -> xyz=0 0 0.4 rpy=0 0 3.1416; parent link1 -> base
